Commit message: added lidar

File: ackermann_vehicle_description/urdf/trooper.urdf.xacro (robot description, xacro)
@@ -299,7 +299,7 @@
                  lr_reflect="${lr_reflect}"/>
   </xacro:macro>
-  <!-- base_footprint must have geometry so that its axes can be displayed in
+  <!-- base_link must have geometry so that its axes can be displayed in
        rviz. -->
-  <link name="base_footprint">
+  <link name="base_link">
     <visual>
       <geometry>
@@ -309,5 +309,5 @@
     </visual>
   </link>
-  <gazebo reference="base_footprint">
+  <gazebo reference="base_link">
     <material>Gazebo/Grey</material>
   </gazebo>
@@ -336,6 +336,6 @@
     <material>Gazebo/Grey</material>
   </gazebo>
-  <joint name="base_footprint_to_chasis" type="fixed">
-    <parent link="base_footprint"/>
+  <joint name="base_link_to_chasis" type="fixed">
+    <parent link="base_link"/>
     <child link="base_link"/>
   </joint>
@@ -356,5 +356,5 @@
     <axis xyz="0 1 0" />
     <origin xyz="0 0 0.3" rpy="0 0 0"/>
-    <parent link="base_footprint"/>
+    <parent link="base_link"/>
     <child link="camera_link"/>
   </joint>

File: ackermann_vehicle_description/urdf/trooper_camera_imu.urdf.xacro (robot description, xacro)
@@ -471,3 +471,64 @@
    </gazebo>
   -->
+<!-- https://answers.ros.org/question/230603/create-a-laser-in-xacro/ -->
+<xacro:laser name="laser_link" parent="base_footprint" xyz="0 0 0" rpy="0 0 0"/>
+<xacro:macro name="laser" params="name parent xyz rpy" >
+  <joint name="${parent}_${name}_joint" type="fixed">
+      <axis xyz="0 0 1" />
+      <origin xyz="${xyz}" rpy="${rpy}"/>
+      <parent link="${parent}"/>
+      <child link="${name}"/>
+    </joint>
+    <link name="${name}">
+      <collision>
+        <origin xyz="0 0 0" rpy="0 0 0"/>
+        <geometry>
+          <box size="0.1 0.1 0.1"/>
+        </geometry>
+      </collision>
+      <visual>
+        <origin xyz="0 0 0" rpy="0 0 0"/>
+        <geometry>
+			    <mesh filename="package://ackermann_vehicle_gazebo/meshes/hokuyo.dae"/>
+        </geometry>
+      </visual>
+      <inertial>
+        <mass value="1e-5" />
+        <origin xyz="0 0 0" rpy="0 0 0"/>
+        <inertia ixx="1e-6" ixy="0" ixz="0" iyy="1e-6" iyz="0" izz="1e-6" />
+      </inertial>
+    </link>
+    <gazebo reference="${name}">
+        <sensor name="laser" type="ray">
+        <pose>0 0 0 0 0 0</pose>
+          <ray>
+            <scan>
+              <horizontal>
+                <!-- The URG-04LX-UG01  has  683 steps with 0.35139 Degree resolution -->
+                <resolution>1</resolution>
+                <max_angle>2.0944</max_angle> <!-- 120 Degree -->
+                <min_angle>-2.0944</min_angle> <!-- -120 Degree -->
+                <samples>683</samples>
+              </horizontal>
+            </scan>
+            <range>
+              <min>0.08</min>
+              <max>5</max>
+              <resolution>0.01</resolution>
+            </range>
+          </ray>
+          <plugin name="laser" filename="libgazebo_ros_laser.so" >
+            <robotNamespace></robotNamespace>
+            <topicName>${name}/scan</topicName>
+            <frameName>${name}</frameName>
+          </plugin>
+          <!--
+          <plugin name="laser" filename="libRayPlugin.so" />
+          -->
+          <always_on>1</always_on>
+          <update_rate>30</update_rate>
+          <visualize>true</visualize>
+        </sensor>
+    </gazebo>
+</xacro:macro>
 </robot>
